File: revA/magstock2018A.kicad_pcb (KiCad board)
At the start: 2 copper layers, 36 parts, among them J1 Audio In, J2 5vdcIn, J3 WS2813, P1 USBMicroB-10118194-0001LF, SW1 TACTILE, SW2 TACTILE, SW3 TACTILE, SW4 TACTILE, SW5 TACTILE, SW6 TACTILE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

Commit message: Update files
Parts:
- removed the REF** at (131.8, 67.1)
- added J4: WS2813, Molex_KK-6410-04_04x2.54mm_Straight, F.Cu at (0.00, 0.00)
- added P2: CONN_1, WagonBG, F.Cu at (134.7, 65.7)
- added REF**: MountingHole_8.4mm_M8_Pad, Mounting_Holes:MountingHole_8.4mm_M8_Pad, F.Cu at (173.3, 41.0)
- moved R3 59.9 mm to (137.3, 82.6), turned to 0 degrees
- moved D5 31.1 mm to (150.0, 78.7), turned to 315 degrees
- moved P1 29.6 mm to (170.2, 78.6)
- moved MK1 27.5 mm to (115.9, 79.7), turned to 90 degrees
- moved C3 25.4 mm to (110.8, 64.9), turned to 135 degrees
- moved R1 24.9 mm to (112.8, 61.4), turned to 120 degrees
- moved D8 21.9 mm to (165.5, 48.6), turned to 135 degrees
- moved J1 21.7 mm to (97.5, 73.6), turned to 34 degrees
- moved R5 21.4 mm to (128.0, 76.2)
- moved C2 21.3 mm to (108.9, 62.0), turned to 225 degrees
- moved U2 20.2 mm to (118.9, 53.6)
- moved J3 19.8 mm to (176.2, 51.4), turned to 248 degrees
- moved J2 19.6 mm to (174.4, 68.7)
- moved C1 19.4 mm to (113.5, 65.7), turned to 90 degrees
- moved R6 18.7 mm to (149.7, 69.9), turned to 315 degrees
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Connections:
- D5 pad 2: Net-(D5-Pad2) -> TUSB
- D7 pad 2: (no net) -> VCC
- D7 pad 3: (no net) -> Net-(D7-Pad3)
- D7 pad 5: (no net) -> GND
- D7 pad 6: (no net) -> Net-(D4-Pad3)
- D8 pad 4: Net-(D8-Pad4) -> Net-(D7-Pad3)
- D9 pad 6: Net-(D8-Pad4) -> Net-(D7-Pad3)
- ESP1 pad 22: (no net) -> TXD
- J2 pad 2: Net-(D5-Pad2) -> VCC
- P1 pad 1: VCC -> TUSB
- P1 pad 2: (no net) -> Net-(P1-Pad2)
- P1 pad 3: (no net) -> Net-(P1-Pad3)
- R6 pad 2: (no net) -> Net-(R6-Pad2)
Routing:
- net VCC: track 0.00 -> 100.7 mm, vias 0 -> 8
- net GND: track 0.00 -> 51.9 mm, vias 0 -> 2
- net +3V3: track 0.00 -> 28.5 mm
- net TUSB: track 0.00 -> 16.3 mm
- net Net-(ESP1-Pad17): track 0.00 -> 15.8 mm
- net Net-(C3-Pad1): track 0.00 -> 12.1 mm
- net ANALOG: track 0.00 -> 11.8 mm
- net Net-(ESP1-Pad1): track 0.00 -> 10.5 mm, vias 0 -> 2
- net Net-(D1-Pad3): track 0.00 -> 10.2 mm
- net RXD: track 0.00 -> 8.53 mm
- net Net-(C1-Pad1): track 0.00 -> 7.49 mm, vias 0 -> 2
Other:
- board outline added: 95.8 x 76.2 mm
- net class Thin added: clearance 0.19558, trace_width 0.254, via_dia 0.6, via_drill 0.4
- net class thick added: clearance 0.19558, trace_width 1.143, via_dia 0.6, via_drill 0.4
- board text added: "120DPI"

Commit message: Update reva
Parts:
- J4: value WS2813 -> Conn_01x05
- R6: value 10k -> 1.5k
- moved J4 142.3 mm to (134.6, 46.3), turned to 270 degrees
- moved C6 20.6 mm to (119.2, 48.6), turned to 90 degrees
- moved D8 12.5 mm to (161.1, 36.9), turned to 168 degrees
- moved D9 12.1 mm to (165.6, 48.2), turned to 135 degrees
- moved REF** 1.41 mm to (174.7, 40.9)
Connections:
- ESP1 pad 19: Net-(ESP1-Pad19) -> D-
- ESP1 pad 20: Net-(ESP1-Pad20) -> D+
- ESP1 pad 6: (no net) -> Net-(ESP1-Pad6)
- J4 pad 1: (no net) -> GND
- J4 pad 2: (no net) -> RXD
- J4 pad 3: (no net) -> TXD
- J4 pad 4: (no net) -> VCC
- P1 pad 2: Net-(P1-Pad2) -> D-
- P1 pad 3: Net-(P1-Pad3) -> D+
- R6 pad 1: RXD -> +3V3
- R6 pad 2: Net-(R6-Pad2) -> D-
- SW2 pad 1: Net-(ESP1-Pad7) -> Net-(ESP1-Pad6)
- SW4 pad 1: Net-(ESP1-Pad18) -> Net-(ESP1-Pad7)
- SW5 pad 1: Net-(ESP1-Pad19) -> Net-(ESP1-Pad17)
- SW6 pad 1: Net-(ESP1-Pad20) -> Net-(ESP1-Pad18)
Routing:
- net GND: track 51.9 -> 333.8 mm, vias 2 -> 16
- net VCC: track 100.7 -> 223.1 mm, vias 8 -> 15
- net D-: track 0.00 -> 87.7 mm, vias 0 -> 2
- net D+: track 0.00 -> 87.5 mm, vias 0 -> 2
- net Net-(ESP1-Pad18): track 0.00 -> 87.5 mm, vias 0 -> 2
- net +3V3: track 28.5 -> 113.8 mm, vias 0 -> 6
- net Net-(ESP1-Pad17): track 15.8 -> 87.7 mm, vias 0 -> 4
- net Net-(ESP1-Pad6): track 0.00 -> 71.1 mm, vias 0 -> 2
- net Net-(ESP1-Pad16): track 0.00 -> 65.5 mm, vias 0 -> 4
- net TXD: track 0.00 -> 51.0 mm, vias 0 -> 2
- net Net-(ESP1-Pad7): track 0.00 -> 50.0 mm, vias 0 -> 4
- net RXD: track 8.53 -> 55.6 mm, vias 0 -> 2
- net Net-(ESP1-Pad5): track 0.00 -> 37.7 mm, vias 0 -> 2
- net Net-(D8-Pad3): track 0.00 -> 24.8 mm, vias 0 -> 2
- net Net-(D4-Pad3): track 0.00 -> 21.9 mm
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Other:
- net class Default: clearance 0.254 -> 0.249
- net class thick: clearance 0.19558 -> 0.29558
- rule trace_clearance: 0.254 -> 0.249
- board text added: "95x76mm"
- board text added: "MAGStock Prototype Board Rev A"

Commit message: Updates!
Routing:
- net (no net): track 0.00 -> 10.4 mm
Changed lines of the file:
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@@
     (area 20.964285 19.245 214.44 104.68565)
     (thickness 1.6)
-    (drawings 4)
-    (tracks 436)
+    (drawings 20)
+    (tracks 450)
     (zones 0)
     (modules 38)
@@
     )
   )
-  (gr_text "MAGStock Prototype Board Rev A" (at 151.915 59.235) (layer B.SilkS)
+  (gr_line (start 105.156 70.612) (end 106.172 70.612) (angle 90) (layer B.SilkS) (width 0.2))
+  (gr_line (start 104.648 71.12) (end 105.156 70.612) (angle 90) (layer B.SilkS) (width 0.2))
+  (gr_line (start 104.648 71.628) (end 104.648 71.12) (angle 90) (layer B.SilkS) (width 0.2))
+  (gr_line (start 105.156 71.628) (end 104.648 71.628) (angle 90) (layer B.SilkS) (width 0.2))
+  (gr_line (start 105.664 71.12) (end 105.156 71.628) (angle 90) (layer B.SilkS) (width 0.2))
+  (gr_line (start 105.664 70.104) (end 105.664 71.12) (angle 90) (layer B.SilkS) (width 0.2))
+  (gr_line (start 106.172 70.612) (end 105.664 70.104) (angle 90) (layer B.SilkS) (width 0.2))
+  (gr_line (start 105.156 71.628) (end 104.648 71.628) (angle 90) (layer F.SilkS) (width 0.2))
+  (gr_line (start 105.664 71.12) (end 105.156 71.628) (angle 90) (layer F.SilkS) (width 0.2))
+  (gr_line (start 105.664 70.612) (end 105.664 71.12) (angle 90) (layer F.SilkS) (width 0.2))
+  (gr_line (start 106.172 70.612) (end 105.664 70.612) (angle 90) (layer F.SilkS) (width 0.2))
+  (gr_line (start 105.664 70.104) (end 106.172 70.612) (angle 90) (layer F.SilkS) (width 0.2))
+  (gr_line (start 105.664 70.612) (end 105.664 70.104) (angle 90) (layer F.SilkS) (width 0.2))
+  (gr_line (start 105.156 70.612) (end 105.664 70.612) (angle 90) (layer F.SilkS) (width 0.2))
+  (gr_line (start 104.648 71.12) (end 105.156 70.612) (angle 90) (layer F.SilkS) (width 0.2))
+  (gr_line (start 104.648 71.628) (end 104.648 71.12) (angle 90) (layer F.SilkS) (width 0.2))
+  (gr_text "MAGStock Prototype Board Rev A" (at 137.575 68.51) (layer B.SilkS)
     (effects (font (size 1.5 1.5) (thickness 0.3)) (justify mirror))
   )
@@
     (effects (font (size 1.5 1.5) (thickness 0.3)))
   )
+  (segment (start 105.664 71.12) (end 105.664 70.104) (width 0.381) (layer B.Cu) (net 0))
+  (segment (start 105.664 70.104) (end 106.172 70.612) (width 0.381) (layer B.Cu) (net 0))
+  (segment (start 106.172 70.612) (end 105.156 70.612) (width 0.381) (layer B.Cu) (net 0))
+  (segment (start 105.156 70.612) (end 104.648 71.12) (width 0.381) (layer B.Cu) (net 0))
+  (segment (start 104.648 71.12) (end 104.648 71.628) (width 0.381) (layer B.Cu) (net 0))
+  (segment (start 104.648 71.628) (end 105.156 71.628) (width 0.381) (layer B.Cu) (net 0))
+  (segment (start 105.156 71.628) (end 105.664 71.12) (width 0.381) (layer B.Cu) (net 0))
+  (segment (start 105.156 71.628) (end 105.664 71.12) (width 0.381) (layer F.Cu) (net 0))
+  (segment (start 105.664 71.12) (end 105.664 70.104) (width 0.381) (layer F.Cu) (net 0))
+  (segment (start 105.664 70.104) (end 106.172 70.612) (width 0.381) (layer F.Cu) (net 0))
+  (segment (start 106.172 70.612) (end 105.156 70.612) (width 0.381) (layer F.Cu) (net 0))
+  (segment (start 105.156 70.612) (end 104.648 71.12) (width 0.381) (layer F.Cu) (net 0))
+  (segment (start 104.648 71.12) (end 104.648 71.628) (width 0.381) (layer F.Cu) (net 0))
+  (segment (start 104.648 71.628) (end 105.156 71.628) (width 0.381) (layer F.Cu) (net 0))
   (segment (start 116.02 66.32) (end 116.96 69.84) (width 0.381) (layer F.Cu) (net 1))
   (segment (start 113.46 66.66) (end 113.44 66.02) (width 0.381) (layer F.Cu) (net 1))

Commit message: Update!
Parts:
- P2: value CONN_1 -> LOGO; footprint WagonBG -> LOGO
Other:
- board text added: "Don't get dysentery."
- board text removed: "MAGStock Prototype Board Rev A"
